File: eagle/main.brd (EAGLE design)
At the start: 73 x 41.3 mm, 24 parts, among them IC1 74LS595D, IC3 317EMP, IC4 74LS595D, Q1 BSS123, Q2 BSS123, Q3 BSS123, Q4 BSS123, Q5 BSS123

Commit message: Temperature control is working.
Parts:
- added C5: 470nF, rcl:C0603K
Connections:
- net GND: now also C5.1
- net N$31: now also C5.2
Routing:
- net N$31: track 2.67 -> 8.13 mm
Other:
- board text added: "FUSERATOR V6"
- board text removed: "FUSERATOR V5"
Changed lines of the file:
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@@
 <layer number="43" name="vRestrict" color="2" fill="10" visible="no" active="yes"/>
 <layer number="44" name="Drills" color="7" fill="1" visible="no" active="yes"/>
-<layer number="45" name="Holes" color="7" fill="1" visible="yes" active="yes"/>
+<layer number="45" name="Holes" color="7" fill="1" visible="no" active="yes"/>
 <layer number="46" name="Milling" color="3" fill="1" visible="no" active="yes"/>
 <layer number="47" name="Measures" color="7" fill="1" visible="no" active="yes"/>
@@
 <layer number="122" name="_bsilk" color="7" fill="1" visible="no" active="yes"/>
 <layer number="151" name="HeatSink" color="7" fill="1" visible="no" active="yes"/>
-<layer number="200" name="200bmp" color="1" fill="10" visible="no" active="yes"/>
+<layer number="200" name="200bmp" color="1" fill="10" visible="yes" active="yes"/>
 <layer number="201" name="201bmp" color="2" fill="10" visible="no" active="yes"/>
 <layer number="202" name="202bmp" color="3" fill="10" visible="no" active="yes"/>
@@
 <hole x="3.175" y="38.1" drill="3.302"/>
 <hole x="3.175" y="3.175" drill="3.302"/>
-<text x="67.31" y="38.1" size="1.27" layer="42" font="vector" ratio="16" rot="MR0" align="center-left">FUSERATOR V5</text>
-<text x="67.31" y="35.56" size="1.27" layer="42" font="vector" ratio="16" rot="MR0" align="center-left">2012 Matthew Gardeski</text>
+<text x="67.31" y="38.1" size="1.27" layer="42" font="vector" ratio="20" rot="MR0" align="center-left">FUSERATOR V6</text>
+<text x="67.31" y="35.56" size="1.27" layer="42" font="vector" ratio="20" rot="MR0" align="center-left">2012 Matthew Gardeski</text>
+<polygon width="0.4064" layer="42">
+<vertex x="23.1775" y="6.6675"/>
+<vertex x="23.1775" y="8.5725"/>
+<vertex x="25.7175" y="8.5725"/>
+<vertex x="25.7175" y="9.2075"/>
+<vertex x="31.115" y="9.2075"/>
+<vertex x="31.115" y="12.065"/>
+<vertex x="32.0675" y="13.0175"/>
+<vertex x="43.815" y="13.0175"/>
+<vertex x="46.0375" y="10.16"/>
+<vertex x="54.61" y="10.16"/>
+<vertex x="54.61" y="5.3975"/>
+<vertex x="53.975" y="4.7625"/>
+<vertex x="20.6375" y="4.7625"/>
+<vertex x="20.6375" y="6.6675"/>
+</polygon>
+<polygon width="0.254" layer="42">
+<vertex x="18.415" y="28.41625"/>
+<vertex x="18.415" y="22.38375"/>
+<vertex x="20.79625" y="22.38375"/>
+<vertex x="20.79625" y="28.41625"/>
+</polygon>
+<polygon width="0.254" layer="42">
+<vertex x="19.52625" y="9.04875"/>
+<vertex x="19.52625" y="19.05"/>
+<vertex x="15.875" y="19.05"/>
+<vertex x="15.875" y="8.89"/>
+<vertex x="19.52625" y="8.89"/>
+</polygon>
+<polygon width="0.254" layer="42">
+<vertex x="18.57375" y="2.54"/>
+<vertex x="18.57375" y="1.905"/>
+<vertex x="54.61" y="1.905"/>
+<vertex x="53.975" y="2.54"/>
+<vertex x="51.59375" y="2.54"/>
+</polygon>
 </plain>
 <attributes>
@@
 <element name="C4" library="rcl" package="E2,5-7" value="" x="50.8" y="11.43" rot="R90"/>
 <element name="J2" library="con-amp" package="10X02MTA" value="" x="24.765" y="9.8425" rot="R270"/>
+<element name="C5" library="rcl" package="C0603K" value="470nF" x="28.73375" y="9.04875" rot="MR225"/>
 </elements>
 <signals>
@@
 <contactref element="430" pad="13"/>
 <contactref element="J2" pad="2"/>
+<contactref element="C5" pad="1"/>
 </signal>
 <signal name="N$17">
@@
 <contactref element="R3" pad="1"/>
 <contactref element="430" pad="11"/>
-<wire x1="31.4325" y1="12.065" x2="31.4325" y2="9.845" width="0.4064" layer="16"/>
-<wire x1="31.4325" y1="9.845" x2="31.7525" y2="9.525" width="0.4064" layer="16"/>
+<wire x1="31.4325" y1="12.065" x2="31.4325" y2="10.1625" width="0.4064" layer="16"/>
+<wire x1="31.4325" y1="10.1625" x2="31.7525" y2="9.525" width="0.4064" layer="16"/>
 <contactref element="J2" pad="1"/>
-<wire x1="24.765" y1="8.5725" x2="28.2575" y2="8.5725" width="0.254" layer="16"/>
-<wire x1="28.2575" y1="8.5725" x2="29.21" y2="9.525" width="0.254" layer="16"/>
-<wire x1="29.21" y1="9.525" x2="31.7525" y2="9.525" width="0.254" layer="16"/>
+<wire x1="31.7525" y1="9.525" x2="29.21" y2="9.525" width="0.254" layer="16"/>
+<wire x1="29.21" y1="9.525" x2="28.2575" y2="8.5725" width="0.2032" layer="16"/>
+<wire x1="28.2575" y1="8.5725" x2="24.765" y2="8.5725" width="0.254" layer="16"/>
 <wire x1="31.4325" y1="12.065" x2="67.31" y2="33.02" width="0" layer="19" extent="1-1"/>
 </signal>
@@
 <wire x1="33.9725" y1="12.065" x2="33.9725" y2="9.845" width="0.4064" layer="16"/>
 <wire x1="33.9725" y1="9.845" x2="33.6525" y2="9.525" width="0.4064" layer="16"/>
+<contactref element="C5" pad="2"/>
+<wire x1="33.6525" y1="9.525" x2="33.6525" y2="8.57" width="0.254" layer="16"/>
+<wire x1="33.6525" y1="8.57" x2="33.3375" y2="8.255" width="0.254" layer="16"/>
+<wire x1="33.3375" y1="8.255" x2="29.5275" y2="8.255" width="0.254" layer="16"/>
+<wire x1="29.5275" y1="8.255" x2="29.35246875" y2="8.43003125" width="0.254" layer="16"/>
 </signal>
 <signal name="N$27">

Commit message: Tidied up the swath of damage i put in last night.
Routing:
- net VCC: track 92.6 -> 105.3 mm
- added copper zone on layer 16, net VCC
Changed lines of the file:
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@@
 <wire x1="2.54" y1="17.61" x2="2.54" y2="25.4" width="0.254" layer="16"/>
 <wire x1="2.54" y1="25.4" x2="15.5575" y2="38.4175" width="0.254" layer="16"/>
-<wire x1="15.5575" y1="38.4175" x2="38.57625" y2="38.4175" width="0.254" layer="16"/>
-<wire x1="38.57625" y1="38.4175" x2="40.3225" y2="36.67125" width="0.254" layer="16"/>
-<wire x1="40.3225" y1="36.67125" x2="40.3225" y2="35.433" width="0.254" layer="16"/>
+<wire x1="15.5575" y1="38.4175" x2="39.0525" y2="38.4175" width="0.254" layer="16"/>
+<wire x1="39.0525" y1="38.4175" x2="40.3225" y2="37.1475" width="0.254" layer="16"/>
+<wire x1="40.3225" y1="37.1475" x2="40.3225" y2="35.433" width="0.254" layer="16"/>
 </signal>
 <signal name="N$10">
@@
 <contactref element="IC3" pad="4"/>
 <contactref element="430" pad="1"/>
-<wire x1="58.01975" y1="10.16" x2="58.89625" y2="11.354" width="0.254" layer="16"/>
+<wire x1="58.33725" y1="11.43" x2="58.89625" y2="11.354" width="0.254" layer="16"/>
 <contactref element="C4" pad="+"/>
 <wire x1="44.1325" y1="12.065" x2="46.0375" y2="10.16" width="0.4064" layer="16"/>
 <wire x1="46.0375" y1="10.16" x2="50.8" y2="10.16" width="0.4064" layer="16"/>
-<wire x1="58.01975" y1="10.16" x2="54.9275" y2="10.16" width="0.4064" layer="16"/>
+<wire x1="58.33725" y1="11.43" x2="57.785" y2="11.43" width="1.27" layer="16"/>
+<wire x1="57.15" y1="11.43" x2="55.88" y2="11.43" width="1.27" layer="16"/>
+<wire x1="55.88" y1="11.43" x2="54.61" y2="10.16" width="1.27" layer="16"/>
 <contactref element="IC4" pad="10"/>
 <contactref element="IC1" pad="10"/>
@@
 <contactref element="C2" pad="2"/>
 <contactref element="C3" pad="2"/>
-<wire x1="54.9275" y1="10.16" x2="50.8" y2="10.16" width="0.4064" layer="16"/>
+<wire x1="54.61" y1="10.16" x2="50.8" y2="10.16" width="1.27" layer="16"/>
 <wire x1="23.8125" y1="4.68125" x2="36.5125" y2="4.68125" width="0.4064" layer="16"/>
 <wire x1="36.5125" y1="4.68125" x2="49.2125" y2="4.68125" width="0.4064" layer="16"/>
@@
 <wire x1="54.0525" y1="4.68125" x2="54.76875" y2="5.3975" width="0.4064" layer="16"/>
 <wire x1="54.76875" y1="5.3975" x2="54.76875" y2="10.00125" width="0.4064" layer="16"/>
-<wire x1="54.76875" y1="10.00125" x2="54.9275" y2="10.16" width="0.254" layer="16"/>
+<wire x1="54.76875" y1="10.00125" x2="54.61" y2="10.16" width="0.254" layer="16"/>
 <wire x1="18.25625" y1="17.145" x2="20.8534" y2="17.145" width="0.254" layer="16"/>
 <wire x1="21.0566" y1="22.225" x2="18.25625" y2="22.225" width="0.254" layer="16"/>
+<wire x1="57.785" y1="11.43" x2="57.785" y2="15.875" width="1.27" layer="16"/>
+<wire x1="57.785" y1="15.875" x2="60.0075" y2="15.875" width="1.27" layer="16"/>
+<wire x1="60.0075" y1="15.875" x2="60.0075" y2="11.43" width="1.27" layer="16"/>
+<wire x1="60.0075" y1="11.43" x2="58.33725" y2="11.43" width="1.27" layer="16"/>
+<wire x1="57.785" y1="11.43" x2="57.15" y2="11.43" width="1.27" layer="16"/>
+<polygon width="0.254" layer="16">
+<vertex x="57.785" y="15.875"/>
+<vertex x="57.785" y="11.43"/>
+<vertex x="60.0075" y="11.43"/>
+<vertex x="60.0075" y="15.875"/>
+<vertex x="57.94375" y="15.875"/>
+</polygon>
 </signal>
 <signal name="GND">
@@
 <contactref element="R4" pad="1"/>
 <contactref element="430" pad="12"/>
-<wire x1="25.615" y1="17.145" x2="30.7975" y2="17.145" width="0.4064" layer="16"/>
-<wire x1="30.7975" y1="17.145" x2="31.4325" y2="16.51" width="0.4064" layer="16"/>
-<wire x1="31.4325" y1="16.51" x2="31.4325" y2="14.605" width="0.4064" layer="16"/>
+<wire x1="25.615" y1="17.145" x2="30.7975" y2="17.145" width="0.254" layer="16"/>
+<wire x1="30.7975" y1="17.145" x2="31.4325" y2="16.51" width="0.254" layer="16"/>
+<wire x1="31.4325" y1="16.51" x2="31.4325" y2="14.605" width="0.254" layer="16"/>
 </signal>
 <signal name="N$30">
